File: Dijous_D_Combustible.kicad_pcb (KiCad board)
At the start: 2 copper layers, 87.6 x 72.4 mm, 64 parts, among them J1 Screw_Terminal_01x02, J2 Conn_01x02, J3 Conn_02x03_Counter_Clockwise, J4 DE9_Plug, J5 Conn_01x02, J6 Conn_01x02, J7 Conn_01x02, K1 Fujitsu_FTR-LYAA005x, K2 Fujitsu_FTR-LYAA005x, Q1 2SC4213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

Commit message: fora grounds de resistències
Routing:
- net GND: track 56.0 -> 44.2 mm, vias 38 -> 30
Changed lines of the file:
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@@
 		(fp_arc
 			(start 12.459619 4.247837)
-			(mid 11.912389 5.195675)
+			(mid 11.912388 5.195671)
 			(end 10.883927 5.57)
 			(stroke
@@
 	)
 	(segment
-		(start 173.736 75.438)
-		(end 174.117 75.438)
-		(width 0.2)
-		(layer "F.Cu")
-		(net 2)
-	)
-	(segment
-		(start 139.7 75.438)
-		(end 139.7 76.9005)
-		(width 0.2)
-		(layer "F.Cu")
-		(net 2)
-	)
-	(segment
 		(start 189.75 90.75)
 		(end 188.4625 90.75)
@@
 	)
 	(segment
-		(start 184.023 101.346)
-		(end 184.023 102.9355)
-		(width 0.2)
-		(layer "F.Cu")
-		(net 2)
-	)
-	(segment
 		(start 139.7 76.9005)
 		(end 139.8885 77.089)
@@
 	)
 	(segment
-		(start 188.4625 90.75)
-		(end 188.4625 89.2875)
-		(width 0.2)
-		(layer "F.Cu")
-		(net 2)
-	)
-	(segment
 		(start 166.5 100.65)
 		(end 166.35 100.5)
@@
 	)
 	(segment
-		(start 174.498 72.517)
-		(end 174.498 73.673)
-		(width 0.2)
-		(layer "F.Cu")
-		(net 2)
-	)
-	(segment
 		(start 185.293 103.124)
 		(end 184.0885 103.124)
@@
 	)
 	(segment
-		(start 188.5 92.25)
-		(end 188.5 90.7875)
-		(width 0.2)
-		(layer "F.Cu")
-		(net 2)
-	)
-	(segment
 		(start 166.5 100.35)
 		(end 166.35 100.5)
@@
 	)
 	(segment
-		(start 139.827 78.74)
-		(end 139.827 77.1505)
-		(width 0.2)
-		(layer "F.Cu")
-		(net 2)
-	)
-	(segment
 		(start 181.0875 81.28)
 		(end 180.955 81.1475)
@@
 	)
 	(segment
-		(start 188.4625 89.2875)
-		(end 188.5 89.25)
-		(width 0.2)
-		(layer "F.Cu")
-		(net 2)
-	)
-	(segment
 		(start 190.435 86)
 		(end 190.105 85.67)
@@
 	)
 	(segment
-		(start 184.023 104.648)
-		(end 184.023 103.0585)
-		(width 0.2)
-		(layer "F.Cu")
-		(net 2)
-	)
-	(segment
-		(start 174.117 75.438)
-		(end 174.825 74.73)
-		(width 0.2)
-		(layer "F.Cu")
-		(net 2)
-	)
-	(segment
 		(start 153.6165 101.5)
 		(end 153.4625 101.346)
@@
 	)
 	(via
-		(at 188.5 92.25)
-		(size 0.6)
-		(drill 0.3)
-		(layers "F.Cu" "B.Cu")
-		(free yes)
-		(net 2)
-	)
-	(via
 		(at 190.25 87.75)
 		(size 0.6)
@@
 	)
 	(via
-		(at 139.827 78.74)
-		(size 0.6)
-		(drill 0.3)
-		(layers "F.Cu" "B.Cu")
-		(free yes)
-		(net 2)
-	)
-	(via
 		(at 170.25 104.14)
 		(size 0.6)
@@
 	)
 	(via
-		(at 184.023 104.648)
-		(size 0.6)
-		(drill 0.3)
-		(layers "F.Cu" "B.Cu")
-		(free yes)
-		(net 2)
-	)
-	(via
 		(at 155 101.5)
 		(size 0.6)
@@
 	)
 	(via
-		(at 188.5 89.25)
-		(size 0.6)
-		(drill 0.3)
-		(layers "F.Cu" "B.Cu")
-		(free yes)
-		(net 2)
-	)
-	(via
-		(at 139.7 75.438)
-		(size 0.6)
-		(drill 0.3)
-		(layers "F.Cu" "B.Cu")
-		(free yes)
-		(net 2)
-	)
-	(via
 		(at 182.626 77.597)
 		(size 0.6)
@@
 	)
 	(via
-		(at 173.736 75.438)
-		(size 0.6)
-		(drill 0.3)
-		(layers "F.Cu" "B.Cu")
-		(free yes)
-		(net 2)
-	)
-	(via
 		(at 168 100.5)
 		(size 0.6)
@@
 	)
 	(via
-		(at 184.023 101.346)
-		(size 0.6)
-		(drill 0.3)
-		(layers "F.Cu" "B.Cu")
-		(free yes)
-		(net 2)
-	)
-	(via
 		(at 161.925 95.758)
 		(size 0.6)
@@
 		(size 0.6)
 		(drill 0.3)
-		(layers "F.Cu" "B.Cu")
-		(free yes)
-		(net 2)
-	)
-	(via
-		(at 174.498 72.517)
-		(size 0.6)
-		(drill 0.3)
