File: Dijous_D_Combustible.kicad_pcb (KiCad board)
At the start: 2 copper layers, 87.6 x 72.4 mm, 64 parts, among them J1 Screw_Terminal_01x02, J2 Conn_01x02, J3 Conn_02x03_Counter_Clockwise, J4 DE9_Plug, J5 Conn_01x02, J6 Conn_01x02, J7 Conn_01x02, K1 Fujitsu_FTR-LYAA005x, K2 Fujitsu_FTR-LYAA005x, Q1 2SC4213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

Commit message: README & LAYOUT & Esquematic
Parts:
- added J8: Conn_01x04, Connector_PinHeader_2.54mm:PinHeader_1x04_P2.54mm_Vertical, F.Cu at (131.5, 80.5)
- added R20: 10k, Resistor_SMD:R_1206_3216Metric, B.Cu at (140.0, 74.0)
- R8: moved to B.Cu
- U2: footprint Package_TO_SOT_SMD:TO-263-5_TabPin3 -> Library:TO-263-5_TabPin3
- U4: footprint Package_TO_SOT_SMD:TO-252-3_TabPin2 -> Library:TO-252-3_TabPin2
- moved R8 0.35 mm to (141.6, 76.9)
Connections:
- U1 pad 1: TXD -> CANTX
- U1 pad 4: RXD -> CANRX
- U3 pad 23: unconnected-(U3A-RB2/CANTX/INT2-Pad23) -> CANRX
- U3 pad 24: unconnected-(U3A-RB3/CANRX-Pad24) -> CANTX
Routing:
- net TXD: track 8.61 -> 39.7 mm, vias 0 -> 2
- net RXD: track 6.01 -> 33.4 mm, vias 0 -> 2
- net GNDPWR: track 60.2 -> 40.7 mm, vias 22 -> 14
- net CANTX: track 0.00 -> 16.5 mm
- net CANRX: track 0.00 -> 14.4 mm
- net GND: track 44.2 -> 48.3 mm, vias 30 -> 33
- net Boto: track 34.1 -> 35.0 mm
- net Retorn_dip: track 24.5 -> 24.0 mm

Commit message: Hola caracola
Parts:
- C7: value 470uF -> 220u
- L1: value 33u -> 68u
- R6: value 3,9K -> 4,7K
Connections:
- R5 pad 2: Vin_Buck -> GND
Changed lines of the file:
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@@
 			)
 		)
-		(property "Value" "3,9K"
+		(property "Value" "4,7K"
 			(at 2.9625 0 -90)
 			(layer "F.Fab")
@@
 		(tags "D2PAK DDPAK TO-263 D2PAK-5 TO-263-5 SOT-426")
 		(property "Reference" "U2"
-			(at -3.707 -6.223 180)
+			(at 0 -6.65 180)
 			(layer "F.SilkS")
 			(effects
@@
 		)
 		(fp_text user "${REFERENCE}"
-			(at 0 3.81 360)
+			(at 0 3.81 0)
 			(layer "F.Fab")
 			(effects
@@
 			)
 		)
-		(property "Value" "33u"
+		(property "Value" "68u"
 			(at 0 1.9 0)
 			(layer "F.Fab")
@@
 			)
 		)
-		(property "Value" "470uF"
+		(property "Value" "220u"
 			(at 0 6.2 90)
 			(layer "F.Fab")
@@
 		(tags "resistor")
 		(property "Reference" "R20"
-			(at 0.1705 -1.864 360)
+			(at 0.1705 -1.864 0)
 			(layer "B.SilkS")
 			(effects
@@
 		)
 		(property "Value" "10k"
-			(at 0 -1.82 360)
+			(at 0 -1.82 0)
 			(layer "B.Fab")
 			(effects
@@
 		)
 		(fp_text user "${REFERENCE}"
-			(at 0 0 360)
+			(at 0 0 0)
 			(layer "B.Fab")
 			(effects
@@
 		(tags "resistor")
 		(property "Reference" "R8"
-			(at -1.607 -2.083 360)
+			(at -1.607 -2.083 0)
 			(layer "B.SilkS")
 			(effects
@@
 		)
 		(property "Value" "4,7k"
-			(at 0 -1.82 360)
+			(at 0 -1.82 0)
 			(layer "B.Fab")
 			(effects
@@
 		)
 		(fp_text user "${REFERENCE}"
-			(at 0 0 360)
+			(at 0 0 0)
 			(layer "B.Fab")
 			(effects
@@
 			(layers "B.Cu" "B.Paste" "B.Mask")
 			(roundrect_rratio 0.222222)
-			(net 57 "Vin_Buck")
+			(net 2 "GND")
 			(pintype "passive")
 		)

Commit message: Layout
Parts:
- D1: value MBR340 -> PMEG040V050EPD; footprint Diode_THT:D_DO-201AD_P15.24mm_Horizontal -> Package_TO_SOT_SMD:Nexperia_CFP15_SOT-1289
- D10, D6, D8, D9: value 1N5408 -> PMEG6030EP; footprint Diode_THT:D_DO-201AD_P15.24mm_Horizontal -> Diode_SMD:D_SOD-128
- J8: value Conn_01x04 -> Conn_01x06; footprint Connector_PinHeader_2.54mm:PinHeader_1x04_P2.54mm_Vertical -> Connector_PinSocket_2.54mm:PinSocket_1x06_P2.54mm_Vertical
- moved D9 55.5 mm to (187.0, 132.0)
- moved R4 38.2 mm to (192.4, 59.0)
- moved J6 32.0 mm to (187.0, 124.5)
- moved D10 28.8 mm to (202.0, 85.8), turned to 90 degrees
- moved D6 24.5 mm to (201.9, 100.3), turned to 90 degrees
- moved D3 17.1 mm to (174.9, 133.1), turned to 0 degrees
- moved J5 15.1 mm to (202.0, 92.0)
- moved J8 13.8 mm to (145.3, 80.8), turned to -90 degrees
- moved D8 13.1 mm to (184.0, 112.0)
- moved R11 13.0 mm to (179.6, 133.1), turned to 180 degrees
- moved D5 10.5 mm to (206.2, 100.6)
- moved R16 9.50 mm to (188.0, 116.0)
- moved REF** 9.34 mm to (204.0, 134.0)
- moved R13 9.29 mm to (206.2, 106.4), turned to 90 degrees
- moved K2 8.58 mm to (197.0, 108.0)
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Connections:
- D1 pad 1: Vin_Buck -> Vbat
- D10 pad 1: Solenoide -> Bomba_combustible
- D9 pad 1: Bomba_combustible -> Solenoide
- J8 pad 2: RXD -> unconnected-(J8-Pin_2-Pad2)
- J8 pad 3: TXD -> +5V
- J8 pad 4: +5V -> TXD
- R5 pad 2: GND -> GNDPWR
Routing:
- net Vin_LDO: track 32.7 -> 3.38 mm, vias 1 -> 0
- net SCL: track 31.8 -> 5.40 mm, vias 2 -> 0
- net Solenoide: track 21.9 -> 5.29 mm
- net R_Dipòsit: track 23.5 -> 11.4 mm, vias 2 -> 1
- net Net-(Q1-B): track 11.6 -> 0.57 mm
- net TXD: track 39.7 -> 29.8 mm, vias 2 -> 0
- net PGC: track 4.70 -> 10.9 mm
- net Vin_Buck: track 19.1 -> 14.1 mm, vias 1 -> 0
- net GND: track 48.3 -> 44.6 mm, vias 33 -> 30
- net Retorn_dip: track 24.0 -> 20.5 mm
- net Nivell_combustible: track 4.88 -> 8.15 mm
- net Net-(Q2-B): track 9.54 -> 7.02 mm
- net Retorn_sol: track 19.9 -> 17.7 mm
- net RXD: track 33.4 -> 31.3 mm, vias 2 -> 0
- net Net-(D7-A): track 2.50 -> 4.01 mm
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- removed copper zone on F.Cu, net +5V
- removed copper zone on B.Cu, net GND
- removed copper zone on B.Cu, net GNDPWR
- removed copper zone on F.Cu, net Vbat
Other:
- board size 87.6 x 72.4 mm -> 80.6 x 67.4 mm

Commit message: Layout+Esquematic+Readme
Parts:
- C8, R14: moved to F.Cu
- R1: moved to B.Cu
- moved R4 51.7 mm to (188.0, 110.5)
- moved D9 44.2 mm to (202.9, 90.8)
- moved J6 43.7 mm to (202.9, 83.8)
- moved D10 30.2 mm to (203.2, 116.0)
- moved J5 30.2 mm to (203.2, 122.2)
- moved D6 25.3 mm to (183.9, 118.1)
- moved R13 24.2 mm to (188.7, 123.1)
- moved D5 24.2 mm to (188.7, 117.3)
- moved D8 22.9 mm to (202.7, 98.8), turned to -90 degrees
- moved R16 16.5 mm to (202.9, 109.0)
- moved D7 14.9 mm to (202.7, 104.1)
- moved Q1 10.2 mm to (190.5, 105.2)
- moved R15 9.96 mm to (184.9, 104.1)
- moved R17 8.51 mm to (182.8, 94.5)
- moved K2 7.15 mm to (194.8, 101.2), turned to 90 degrees
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Connections:
- U3 pad 22: LED_pneumatics -> unconnected-(U3A-RB1/INT1-Pad22)
- U3 pad 6: unconnected-(U3A-RA4/T0CKI-Pad6) -> LED_pneumatics
Routing:
- net SCL: track 5.40 -> 36.3 mm, vias 0 -> 2
- net Vin_LDO: track 3.38 -> 24.8 mm
- net GNDPWR: track 39.9 -> 50.9 mm, vias 13 -> 18
- net TXD: track 29.8 -> 38.8 mm
- net Solenoide: track 5.29 -> 14.1 mm
- net R_Dipòsit: track 11.4 -> 19.0 mm, vias 1 -> 0
- net Retorn_dip: track 20.5 -> 14.2 mm
- net Retorn_sol: track 17.7 -> 22.9 mm
- net GND: track 44.6 -> 48.8 mm, vias 30 -> 51
- net +5V: track 9.82 -> 13.8 mm
- net SCA: track 34.7 -> 38.5 mm
- net Net-(Q2-B): track 7.02 -> 4.26 mm
- net Net-(Q1-B): track 0.57 -> 3.28 mm
- net R_Bomba: track 33.0 -> 35.5 mm, vias 1 -> 0
- net LED_pneumatics: track 21.7 -> 19.1 mm, vias 2 -> 0
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- added copper zone on F.Cu, net +5V
- added copper zone on B.Cu, net GND
- added copper zone on B.Cu, net GNDPWR
- added copper zone on F.Cu, net Vbat

Commit message: Todo
Parts:
- removed R20: 10k, Resistor_SMD:R_1206_3216Metric
- D3: value LED -> LED_Power
- D5, D7: value LED -> LED_Relé
- J2: footprint Connector_PinHeader_2.00mm:PinHeader_2x01_P2.00mm_Vertical -> Connector_PinHeader_2.54mm:PinHeader_1x02_P2.54mm_Vertical
- R11: value 460 -> 330
- R13, R16: value 510 -> 290
Routing:
- net TXD: track 38.8 -> 31.5 mm
- net Boto: track 34.9 -> 37.6 mm, vias 0 -> 1

Commit message: Can transciever
Parts:
- U1: value MCP2551-I-SN -> MCP2557FD-xSN

Commit message: De todo
Parts:
- J8: footprint Connector_PinSocket_2.54mm:PinSocket_1x06_P2.54mm_Vertical -> Connector_PinHeader_2.54mm:PinHeader_1x06_P2.54mm_Vertical
- moved J8 0.77 mm to (144.0, 80.5)
Changed lines of the file:
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@@
 			(outputformat 1)
 			(mirror no)
-			(drillshape 1)
+			(drillshape 0)
 			(scaleselection 1)
-			(outputdirectory "")
+			(outputdirectory "Gerbers/")
 		)
 	)
@@
 		)
 	)
-	(footprint "Connector_PinSocket_2.54mm:PinSocket_1x06_P2.54mm_Vertical"
+	(footprint "Connector_PinHeader_2.54mm:PinHeader_1x06_P2.54mm_Vertical"
 		(layer "F.Cu")
-		(at 144.78 80.645 -90)
-		(descr "Through hole straight socket strip, 1x06, 2.54mm pitch, single row (from Kicad 4.0.7), script generated")
-		(tags "Through hole socket strip THT 1x06 2.54mm single row")
+		(at 144.018 80.518 -90)
+		(descr "Through hole straight pin header, 1x06, 2.54mm pitch, single row")
+		(tags "Through hole pin header THT 1x06 2.54mm single row")
 		(property "Reference" "J8"
-			(at -2.54 -0.762 180)
+			(at 0 -2.33 -90)
 			(layer "F.SilkS")
 			(effects
@@
 		)
 		(property "Value" "Conn_01x06"
-			(at 0 15.47 90)
+			(at 0 15.03 -90)
 			(layer "F.Fab")
 			(effects
@@
 			)
 		)
-		(property "Footprint" "Connector_PinSocket_2.54mm:PinSocket_1x06_P2.54mm_Vertical"
+		(property "Footprint" "Connector_PinHeader_2.54mm:PinHeader_1x06_P2.54mm_Vertical"
 			(at 0 0 -90)
 			(unlocked yes)
@@
 		)
 		(fp_line
-			(start 0 -1.33)
-			(end 1.33 -1.33)
+			(start -1.33 0)
+			(end -1.33 -1.33)
 			(stroke
 				(width 0.12)
@@
 		)
 		(fp_line
-			(start 1.33 -1.33)
-			(end 1.33 0)
+			(start -1.33 -1.33)
+			(end 0 -1.33)
 			(stroke
 				(width 0.12)
@@
 		)
 		(fp_line
-			(start -1.8 14.45)
-			(end -1.8 -1.8)
+			(start -1.8 14.5)
+			(end 1.8 14.5)
 			(stroke
 				(width 0.05)
@@
 		)
 		(fp_line
-			(start 1.75 14.45)
-			(end -1.8 14.45)
+			(start 1.8 14.5)
+			(end 1.8 -1.8)
 			(stroke
 				(width 0.05)
@@
 		(fp_line
 			(start -1.8 -1.8)
-			(end 1.75 -1.8)
+			(end -1.8 14.5)
 			(stroke
 				(width 0.05)
@@
 		)
 		(fp_line
-			(start 1.75 -1.8)
-			(end 1.75 14.45)
+			(start 1.8 -1.8)
+			(end -1.8 -1.8)
 			(stroke
 				(width 0.05)
@@
 		(fp_line
 			(start -1.27 13.97)
-			(end -1.27 -1.27)
+			(end -1.27 -0.635)
 			(stroke
 				(width 0.1)
@@
 		)
 		(fp_line
-			(start 1.27 -0.635)
-			(end 1.27 13.97)
+			(start -1.27 -0.635)
+			(end -0.635 -1.27)
 			(stroke
 				(width 0.1)
@@
 		)
 		(fp_line
-			(start -1.27 -1.27)
-			(end 0.635 -1.27)
+			(start -0.635 -1.27)
+			(end 1.27 -1.27)
 			(stroke
 				(width 0.1)
@@
 		)
 		(fp_line
-			(start 0.635 -1.27)
-			(end 1.27 -0.635)
+			(start 1.27 -1.27)
+			(end 1.27 13.97)
 			(stroke
 				(width 0.1)
@@
 			(pintype "passive+no_connect")
 		)
-		(model "${KICAD8_3DMODEL_DIR}/Connector_PinSocket_2.54mm.3dshapes/PinSocket_1x06_P2.54mm_Vertical.wrl"
+		(model "${KICAD8_3DMODEL_DIR}/Connector_PinHeader_2.54mm.3dshapes/PinHeader_1x06_P2.54mm_Vertical.wrl"
 			(offset
 				(xyz 0 0 0)
@@
 	)
 	(segment
-		(start 160.75 93.9462)
-		(end 160.705 93.9912)
-		(width 0.4)
+		(start 136.398 81.788)
+		(end 144.96 90.35)
+		(width 0.3)
 		(layer "F.Cu")
 		(net 35)
 	)
 	(segment
-		(start 160.705 94.697199)
-		(end 160.705 93.9912)
-		(width 0.2)
+		(start 136.398 80.518)
+		(end 136.398 81.788)
+		(width 0.3)
 		(layer "F.Cu")
 		(net 35)
 	)
 	(segment
-		(start 137.16 80.645)
-		(end 137.16 82.55)
-		(width 0.3)
+		(start 160.75 93.9462)
+		(end 160.705 93.9912)
+		(width 0.4)
 		(layer "F.Cu")
 		(net 35)
 	)
 	(segment
-		(start 160.75 94.0362)
+		(start 160.705 94.697199)
 		(end 160.705 93.9912)
-		(width 0.3)
+		(width 0.2)
 		(layer "F.Cu")
 		(net 35)
 	)
 	(segment
-		(start 137.16 82.55)
-		(end 144.96 90.35)
+		(start 160.75 94.0362)
+		(end 160.705 93.9912)
 		(width 0.3)
 		(layer "F.Cu")
@@
 	)
 	(segment
-		(start 160.705 93.141)
-		(end 160.705 93.9912)
+		(start 144.96 90.35)
+		(end 157.914 90.35)
 		(width 0.3)
 		(layer "F.Cu")
@@
 	)
 	(segment
-		(start 144.96 90.35)
-		(end 157.914 90.35)
+		(start 160.705 93.141)
+		(end 160.705 93.9912)
 		(width 0.3)
 		(layer "F.Cu")
@@
 	)
 	(segment
-		(start 159.435 92.887)
-		(end 159.435 93.9912)
-		(width 0.3)
-		(layer "F.Cu")
-		(net 36)
-	)
-	(segment
-		(start 135.128 81.153)
-		(end 135.128 81.28)
-		(width 0.3)
-		(layer "F.Cu")
-		(net 36)
-	)
-	(segment
-		(start 134.62 80.645)
-		(end 134.62 81.407)
+		(start 133.858 80.645)
+		(end 144.063 90.85)
 		(width 0.3)
 		(layer "F.Cu")
@@
 	)
 	(segment
-		(start 157.398 90.85)
-		(end 159.435 92.887)
+		(start 159.435 92.887)
+		(end 159.435 93.9912)
 		(width 0.3)
 		(layer "F.Cu")
@@
 	)
 	(segment
-		(start 134.62 80.645)
-		(end 135.128 81.153)
+		(start 159.4104 94.0158)
+		(end 159.435 93.9912)
 		(width 0.3)
 		(layer "F.Cu")
@@
 	)
 	(segment
-		(start 159.4104 94.0158)
-		(end 159.435 93.9912)
+		(start 133.858 80.518)
+		(end 133.858 80.645)
 		(width 0.3)
 		(layer "F.Cu")
@@
 	)
 	(segment
-		(start 134.62 81.407)
-		(end 144.063 90.85)
+		(start 157.398 90.85)
+		(end 159.435 92.887)
 		(width 0.3)
 		(layer "F.Cu")
