File: Dijous_D_Combustible.kicad_sch (KiCad schematic)
At the start: 60 parts, among them J1 Screw_Terminal_01x02, J2 Conn_01x02, J3 Conn_02x03_Counter_Clockwise, J4 DE9_Plug, J5 Conn_01x02, J6 Conn_01x02, J7 Conn_01x02, K1 Fujitsu_FTR-LYAA005x, K2 Fujitsu_FTR-LYAA005x, Q1 2SC4213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

Commit message: README & LAYOUT & Esquematic
Parts:
- removed D10, D6: LED, LED_SMD:LED_0805_2012Metric, symbol Device:LED
- removed D4, D5: 1N5408, Diode_THT:D_DO-201AD_P15.24mm_Horizontal, symbol Diode:1N5408
- added D10, D6: 1N5408, Diode_THT:D_DO-201AD_P15.24mm_Horizontal, symbol Diode:1N5408
- added D4, D5: LED, LED_SMD:LED_0805_2012Metric, symbol Device:LED
- added J8: Conn_01x04, Connector_PinHeader_2.54mm:PinHeader_1x04_P2.54mm_Vertical, symbol Connector_Generic:Conn_01x04
- added R20: 10k, Resistor_SMD:R_1206_3216Metric, symbol Device:R
- R10: value 510 -> 10K
- R11: value 4,7k -> 460
- R12: value 1k -> 515
- R13: value 10K -> 510
- R14: value 10K -> 4,7k
- R15: value 460 -> 1k
- R19: value 515 -> 10k; footprint Resistor_SMD:R_1206_3216Metric -> Resistor_SMD:R_0805_2012Metric
- R9: value 10k -> 10K; footprint Resistor_SMD:R_0805_2012Metric -> Resistor_SMD:R_1206_3216Metric
Connections:
- net +5V: now also R10.1, R19.1, J8.4 (Pin_4); no longer R13.1, R14.1
- net Bomba_combustible: now also D9.1 (K), J5.1 (Pin_1); no longer J7.1 (Pin_1)
- net GND: now also J7.2 (Pin_2), R12.2, R14.2, J8.1 (Pin_1), R20.2; no longer J6.2 (Pin_2), R11.2, R19.2
- net GNDPWR: now also D3.1 (K), J6.2 (Pin_2), D10.2 (A); no longer J7.2 (Pin_2)
- net LED_pneumatics: now also D4.2 (A)
- net Nivell_combustible: now also J7.1 (Pin_1); no longer J6.1 (Pin_1)
- net RXD: now also J8.2 (Pin_2); no longer U1.4 (RXD)
- net R_Bomba: now also R14.1, R15.1; no longer R11.1, R12.1
- net Retorn_sol: now also D5.1 (K), D6.2 (A); no longer D3.1 (K)
- net SCA: now also R9.2; no longer R13.2
- net SCL: now also R10.2; no longer R14.2
- net Solenoide: now also J6.1 (Pin_1), D10.1 (K); no longer D9.1 (K), J5.1 (Pin_1)
- net TXD: now also J8.3 (Pin_3), R20.1; no longer U1.1 (TXD)
- net Vbat: now also R11.1, R13.1, D6.1 (K); no longer R10.1, R15.1
- net at R15.2: now also Q1.1 (B)
- net at D3.2 (A): now also R11.2; no longer R10.2
- net at JP1.3 (B), SW1.1: now also R19.2; no longer R9.2
- net CANRX: now reaches U3.23 (RB2/CANTX/INT2)
- net CANRX: now also U1.4 (RXD)
- net CANTX: now reaches U3.24 (RB3/CANRX)
- net CANTX: now also U1.1 (TXD)
- new net: D5.2 (A), R13.2
- new net: D4.1 (K), R12.1
- no-connect marks 21 -> 19
Other:
- note added: "Conector USART"

Commit message: Hola caracola
Parts:
- C7: value 470uF -> 220u
- L1: value 33u -> 68u
- R6: value 3,9K -> 4,7K
- U2: footprint Package_TO_SOT_SMD:TO-263-5_TabPin3 -> Library:TO-263-5_TabPin3
- U4: footprint Package_TO_SOT_SMD:TO-252-3_TabPin2 -> Library:TO-252-3_TabPin2
Connections:
- net GND: now also R5.2
- net Vin_Buck: no longer R5.2
Other:
- moved on the sheet: R5
Changed lines of the file:
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@@
 	)
 	(junction
+		(at 118.11 22.86)
+		(diameter 0)
+		(color 0 0 0 0)
+	)
+	(junction
 		(at 267.97 177.8)
 		(diameter 0)
@@
 	(wire
 		(pts
-			(xy 118.11 22.86) (xy 118.11 34.29)
-		)
-		(stroke
-			(width 0)
-			(type default)
-		)
-	)
-	(wire
-		(pts
 			(xy 349.25 33.02) (xy 349.25 30.48)
 		)
@@
 	(wire
 		(pts
-			(xy 83.82 34.29) (xy 99.06 34.29)
-		)
-		(stroke
-			(width 0)
-			(type default)
-		)
-	)
-	(wire
-		(pts
 			(xy 107.95 166.37) (xy 107.95 158.75)
 		)
@@
 	(wire
 		(pts
+			(xy 118.11 22.86) (xy 118.11 34.29)
+		)
+		(stroke
+			(width 0)
+			(type default)
+		)
+	)
+	(wire
+		(pts
 			(xy 349.25 52.07) (xy 356.87 52.07)
 		)
@@
 	(wire
 		(pts
-			(xy 106.68 34.29) (xy 118.11 34.29)
+			(xy 106.68 22.86) (xy 118.11 22.86)
 		)
 		(stroke
@@
 	(wire
 		(pts
+			(xy 99.06 22.86) (xy 99.06 29.21)
+		)
+		(stroke
+			(width 0)
+			(type default)
+		)
+	)
+	(wire
+		(pts
 			(xy 351.79 127) (xy 351.79 123.19)
 		)
@@
 	(wire
 		(pts
-			(xy 83.82 45.72) (xy 83.82 34.29)
-		)
-		(stroke
-			(width 0)
-			(type default)
-		)
-	)
-	(wire
-		(pts
 			(xy 167.64 50.8) (xy 172.72 50.8)
 		)
@@
 			)
 		)
-		(property "Value" "33u"
+		(property "Value" "68u"
 			(at 135.89 48.26 90)
 			(effects
@@
 			)
 		)
-		(property "Value" "470uF"
+		(property "Value" "220u"
 			(at 148.59 55.8799 0)
 			(effects
@@
 			)
 		)
-		(property "Footprint" "Package_TO_SOT_SMD:TO-263-5_TabPin3"
+		(property "Footprint" "Library:TO-263-5_TabPin3"
 			(at 106.68 54.61 0)
 			(effects
@@
 			)
 		)
-		(property "Value" "3,9K"
+		(property "Value" "4,7K"
 			(at 121.92 30.48 90)
 			(effects
@@
 			)
 		)
-		(property "Footprint" "Package_TO_SOT_SMD:TO-252-3_TabPin2"
+		(property "Footprint" "Library:TO-252-3_TabPin2"
 			(at 180.34 50.8 0)
 			(effects
@@
 	)
 	(symbol
+		(lib_id "power:GND")
+		(at 99.06 29.21 0)
+		(unit 1)
+		(exclude_from_sim no)
+		(in_bom yes)
+		(on_board yes)
+		(dnp no)
+		(fields_autoplaced yes)
+		(property "Reference" "#PWR49"
+			(at 99.06 35.56 0)
+			(effects
+				(font
+					(size 1.27 1.27)
+				)
+				(hide yes)
+			)
+		)
+		(property "Value" "GND"
+			(at 99.06 34.29 0)
+			(effects
+				(font
+					(size 1.27 1.27)
+				)
+			)
+		)
+		(property "Footprint" ""
+			(at 99.06 29.21 0)
+			(effects
+				(font
+					(size 1.27 1.27)
+				)
+				(hide yes)
+			)
+		)
+		(property "Datasheet" ""
+			(at 99.06 29.21 0)
+			(effects
+				(font
+					(size 1.27 1.27)
+				)
+				(hide yes)
+			)
+		)
+		(property "Description" "Power symbol creates a global label with name \"GND\" , ground"
+			(at 99.06 29.21 0)
+			(effects
+				(font
+					(size 1.27 1.27)
+				)
+				(hide yes)
+			)
+		)
+		(pin "1"
+		)
+		(instances
+			(project ""
+				(path "/8e5e5a45-9171-45b6-b00a-10c0ac4f5428"
+					(reference "#PWR49")
+					(unit 1)
+				)
+			)
+		)
+	)
+	(symbol
 		(lib_id "Connector_Generic:Conn_01x04")
 		(at 29.21 107.95 180)
@@
 	(symbol
 		(lib_id "Device:R")
-		(at 102.87 34.29 270)
+		(at 102.87 22.86 270)
 		(unit 1)
 		(exclude_from_sim no)
@@
 		(fields_autoplaced yes)
 		(property "Reference" "R5"
-			(at 102.87 27.94 90)
+			(at 102.87 16.51 90)
 			(effects
 				(font
@@
 		)
 		(property "Value" "1k"
-			(at 102.87 30.48 90)
+			(at 102.87 19.05 90)
 			(effects
 				(font
@@
 		)
 		(property "Footprint" "Resistor_SMD:R_1206_3216Metric"
-			(at 102.87 32.512 90)
+			(at 102.87 21.082 90)
 			(effects
 				(font
@@
 		)
 		(property "Datasheet" "~"
-			(at 102.87 34.29 0)
+			(at 102.87 22.86 0)
 			(effects
 				(font
@@
 		)
 		(property "Description" "Resistor"
-			(at 102.87 34.29 0)
+			(at 102.87 22.86 0)
 			(effects
 				(font

Commit message: Layout
Parts:
- removed D1: MBR340, Diode_THT:D_DO-201AD_P15.24mm_Horizontal, symbol Diode:MBR340
- removed D10, D6, D8, D9: 1N5408, Diode_THT:D_DO-201AD_P15.24mm_Horizontal, symbol Diode:1N5408
- removed J8: Conn_01x04, Connector_PinHeader_2.54mm:PinHeader_1x04_P2.54mm_Vertical, symbol Connector_Generic:Conn_01x04
- removed R20: 10k, Resistor_SMD:R_1206_3216Metric, symbol Device:R
- added D1: PMEG040V050EPD, Package_TO_SOT_SMD:Nexperia_CFP15_SOT-1289, symbol Diode:PMEG040V050EPD
- added D10, D6, D8, D9: PMEG6030EP, Diode_SMD:D_SOD-128, symbol Diode:PMEG6030EP
- added J8: Conn_01x06, Connector_PinSocket_2.54mm:PinSocket_1x06_P2.54mm_Vertical, symbol Connector_Generic:Conn_01x06
Connections:
- net +5V: now also J8.3 (Pin_3)
- net Bomba_combustible: now also D10.1 (K)
- net GND: now also J8.1 (Pin_1); no longer R5.2
- net GNDPWR: now also R5.2, D10.2 (A), D9.2 (A)
- net RXD: now also J8.5 (Pin_5)
- net Retorn_dip: now also D8.2 (A)
- net Retorn_sol: now also D6.2 (A)
- net Solenoide: now also D9.1 (K)
- net TXD: now also J8.4 (Pin_4)
- net Vbat: now also D1.1 (A), D1.2 (A), D6.1 (K), D8.1 (K)
- net Vin_Buck: now also D1.3 (K)
- no-connect marks 19 -> 21
Other:
- moved on the sheet: R5

Commit message: Layout+Esquematic+Readme
Connections:
- net LED_pneumatics: now also U3.6 (RA4/T0CKI); no longer U3.22 (RB1/INT1)
Changed lines of the file:
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@@
+	)
+	(no_connect
+		(at 171.45 147.32)
 	)
 	(no_connect
@@
 	)
 	(no_connect
-		(at 262.89 152.4)
-	)
-	(no_connect
 		(at 262.89 154.94)
 	)
@@
 	(wire
 		(pts
+			(xy 269.24 148.59) (xy 265.43 148.59)
+		)
+		(stroke
+			(width 0)
+			(type default)
+		)
+	)
+	(wire
+		(pts
 			(xy 193.04 191.77) (xy 193.04 194.31)
 		)
@@
 	(wire
 		(pts
+			(xy 265.43 148.59) (xy 265.43 152.4)
+		)
+		(stroke
+			(width 0)
+			(type default)
+		)
+	)
+	(wire
+		(pts
 			(xy 254 55.88) (xy 255.27 55.88)
 		)
@@
 	(wire
 		(pts
+			(xy 265.43 152.4) (xy 262.89 152.4)
+		)
+		(stroke
+			(width 0)
+			(type default)
+		)
+	)
+	(wire
+		(pts
 			(xy 349.25 49.53) (xy 349.25 52.07)
 		)
@@
 		(pts
 			(xy 180.34 191.77) (xy 180.34 194.31)
-		)
-		(stroke
-			(width 0)
-			(type default)
-		)
-	)
-	(wire
-		(pts
-			(xy 157.48 147.32) (xy 171.45 147.32)
 		)
 		(stroke
@@
 	(global_label "LED_pneumatics"
 		(shape output)
-		(at 157.48 147.32 180)
+		(at 269.24 148.59 0)
 		(fields_autoplaced yes)
 		(effects
@@
 				(size 1.27 1.27)
 			)
-			(justify right)
+			(justify left)
 		)
 		(property "Intersheetrefs" "${INTERSHEET_REFS}"
-			(at 139.255 147.32 0)
+			(at 287.465 148.59 0)
 			(effects
 				(font
 					(size 1.27 1.27)
 				)
-				(justify right)
+				(justify left)
 				(hide yes)
 			)

Commit message: Todo
Parts:
- D3: value LED -> LED_Power
- D5, D7: value LED -> LED_Relé
- J2: footprint Connector_PinHeader_2.00mm:PinHeader_2x01_P2.00mm_Vertical -> Connector_PinHeader_2.54mm:PinHeader_1x02_P2.54mm_Vertical
- JP1: now in the parts list
- R11: value 460 -> 330
- R13, R16: value 510 -> 290
Other:
- note added: "LED PNEUMÀTICS = Vermell"
- note added: "LED POWER = Verd"
- note removed: "LED POWER = Vermell"

Commit message: Can transciever
Parts:
- removed U1: MCP2551-I-SN, Package_SO:SOIC-8_3.9x4.9mm_P1.27mm, symbol Interface_CAN_LIN:MCP2551-I-SN
- added U1: MCP2557FD-xSN, Package_SO:SOIC-8_3.9x4.9mm_P1.27mm, symbol Interface_CAN_LIN:MCP2557FD-xSN
Connections:
- net +5V: now also U1.3 (VDD)
- net CANRX: now also U1.4 (RXD)
- net CANTX: now also U1.1 (TXD)
- net Can+: now also U1.7 (CANH)
- net Can-: now also U1.6 (CANL)
- net GND: now also U1.2 (VSS)
- net at R1.1: now also U1.8 (S)
- no-connect marks 21 -> 20
Changed lines of the file:
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@@
 		(at 262.89 160.02)
 	)
-	(no_connect
-		(at 44.45 170.18)
-	)
 	(wire
 		(pts
@@
 	)
 	(global_label "CANRX"
-		(shape input)
+		(shape output)
 		(at 171.45 149.86 180)
 		(fields_autoplaced yes)
@@
 	)
 	(symbol
-		(lib_id "Interface_CAN_LIN:MCP2551-I-SN")
-		(at 57.15 167.64 0)
-		(unit 1)
-		(exclude_from_sim no)
-		(in_bom yes)
-		(on_board yes)
-		(dnp no)
-		(fields_autoplaced yes)
-		(property "Reference" "U1"
-			(at 59.3441 154.94 0)
-			(effects
-				(font
-					(size 1.27 1.27)
-				)
-				(justify left)
-			)
-		)
-		(property "Value" "MCP2551-I-SN"
-			(at 59.3441 157.48 0)
-			(effects
-				(font
-					(size 1.27 1.27)
-				)
-				(justify left)
-			)
-		)
-		(property "Footprint" "Package_SO:SOIC-8_3.9x4.9mm_P1.27mm"
-			(at 57.15 180.34 0)
-			(effects
-				(font
-					(size 1.27 1.27)
-					(italic yes)
-				)
-				(hide yes)
-			)
-		)
-		(property "Datasheet" "http://ww1.microchip.com/downloads/en/devicedoc/21667d.pdf"
-			(at 57.15 167.64 0)
-			(effects
-				(font
-					(size 1.27 1.27)
-				)
-				(hide yes)
-			)
-		)
-		(property "Description" "High-Speed CAN Transceiver, 1Mbps, 5V supply, SOIC-8"
-			(at 57.15 167.64 0)
-			(effects
-				(font
-					(size 1.27 1.27)
-				)
-				(hide yes)
-			)
-		)
-		(property "Sim.Device" ""
-			(at 57.15 167.64 0)
-			(effects
-				(font
-					(size 1.27 1.27)
-				)
-				(hide yes)
-			)
-		)
-		(property "Sim.Pins" ""
-			(at 57.15 167.64 0)
-			(effects
-				(font
-					(size 1.27 1.27)
-				)
-				(hide yes)
-			)
-		)
-		(property "Campo7" ""
-			(at 57.15 167.64 0)
-			(effects
-				(font
-					(size 1.27 1.27)
-				)
-				(hide yes)
-			)
-		)
-		(pin "1"
-		)
-		(pin "2"
-		)
-		(pin "3"
-		)
-		(pin "4"
-		)
-		(pin "5"
-		)
-		(pin "6"
-		)
-		(pin "7"
-		)
-		(pin "8"
-		)
-		(instances
-			(project "Dijous_D_Combustible"
-				(path "/8e5e5a45-9171-45b6-b00a-10c0ac4f5428"
-					(reference "U1")
-					(unit 1)
-				)
-			)
-		)
-	)
-	(symbol
 		(lib_id "power:GNDPWR")
 		(at 273.05 67.31 0)
@@
 					(unit 1)
 				)
+			)
+		)
+	)
+	(symbol
+		(lib_id "Interface_CAN_LIN:MCP2557FD-xSN")
+		(at 57.15 167.64 0)
+		(unit 1)
+		(exclude_from_sim no)
+		(in_bom yes)
+		(on_board yes)
+		(dnp no)
+		(fields_autoplaced yes)
+		(property "Reference" "U1"
+			(at 59.3441 154.94 0)
+			(effects
+				(font
+					(size 1.27 1.27)
+				)
+				(justify left)
+			)
+		)
+		(property "Value" "MCP2557FD-xSN"
+			(at 59.3441 157.48 0)
+			(effects
+				(font
+					(size 1.27 1.27)
+				)
+				(justify left)
+			)
+		)
+		(property "Footprint" "Package_SO:SOIC-8_3.9x4.9mm_P1.27mm"
+			(at 57.15 182.88 0)
+			(effects
+				(font
+					(size 1.27 1.27)
+				)
+				(hide yes)
+			)
+		)
+		(property "Datasheet" "https://ww1.microchip.com/downloads/en/DeviceDoc/20005533A.pdf"
+			(at 57.15 167.64 0)
+			(effects
+				(font
+					(size 1.27 1.27)
+				)
+				(hide yes)
+			)
+		)
+		(property "Description" "CAN FD Transceiver with Silent Mode, up to 8 Mbps, SOIC-8"
+			(at 57.15 167.64 0)
+			(effects
+				(font
+					(size 1.27 1.27)
+				)
+				(hide yes)
+			)
+		)
+		(pin "1"
+		)
+		(pin "2"
+		)
+		(pin "6"
+		)
+		(pin "5"
+		)
+		(pin "3"
+		)
+		(pin "8"
+		)
+		(pin "7"
+		)
+		(pin "4"
+		)
+		(instances
+			(project ""
+				(path "/8e5e5a45-9171-45b6-b00a-10c0ac4f5428"
+					(reference "U1")
+					(unit 1)
+				)

Commit message: De todo
Parts:
- J8: footprint Connector_PinSocket_2.54mm:PinSocket_1x06_P2.54mm_Vertical -> Connector_PinHeader_2.54mm:PinHeader_1x06_P2.54mm_Vertical
Changed lines of the file:
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@@
 			)
 		)
-		(property "Footprint" "Connector_PinSocket_2.54mm:PinSocket_1x06_P2.54mm_Vertical"
+		(property "Footprint" "Connector_PinHeader_2.54mm:PinHeader_1x06_P2.54mm_Vertical"
 			(at 21.59 105.41 0)
 			(effects
